File: Evan-PCB-ISP.kicad_pcb (KiCad board)
At the start: 2 copper layers, 76.2 x 38.1 mm, 24 parts, among them SW1 SW_Push, U1 ATmega32U4-AU, Y1 16MHz

Commit message: Created Gerber Files
Routing:
- net Net-(USB1-Pad6): track 0.00 -> 16.3 mm
Changed lines of the file:
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@@
     (thickness 1.6)
     (drawings 11)
-    (tracks 209)
+    (tracks 213)
     (zones 0)
     (modules 24)
@@
     (solder_mask_min_width 0.25)
     (aux_axis_origin 0 0)
-    (visible_elements FFFFFF7F)
+    (visible_elements 7FFFFFFF)
     (pcbplotparams
-      (layerselection 0x010fc_ffffffff)
-      (usegerberextensions false)
+      (layerselection 0x010f0_ffffffff)
+      (usegerberextensions true)
       (usegerberattributes false)
       (usegerberadvancedattributes false)
@@
       (plotinvisibletext false)
       (padsonsilk false)
-      (subtractmaskfromsilk false)
+      (subtractmaskfromsilk true)
       (outputformat 1)
       (mirror false)
-      (drillshape 1)
+      (drillshape 0)
       (scaleselection 1)
       (outputdirectory ""))
@@
   (segment (start 148.336 106.934) (end 146.939 106.934) (width 0.254) (layer B.Cu) (net 20))
   (segment (start 146.939 106.934) (end 146.65275 106.64775) (width 0.254) (layer B.Cu) (net 20))
+  (segment (start 116.1745 87.812) (end 116.1745 83.312) (width 0.254) (layer B.Cu) (net 43))
+  (segment (start 117.2785 83.312) (end 123.4745 83.312) (width 0.254) (layer B.Cu) (net 43))
+  (segment (start 116.1745 83.312) (end 117.2785 83.312) (width 0.254) (layer B.Cu) (net 43))
+  (segment (start 123.4745 83.312) (end 123.4745 87.812) (width 0.254) (layer B.Cu) (net 43))
   (zone (net 1) (net_name GND) (layer B.Cu) (hatch edge 0.508)
     (connect_pads (clearance 0.508))
