File: Rev 1/Rev 1.sch (KiCad schematic (older format))
At the start: 35 parts, among them U1 nice_nano

Commit message: rev 1 finished
Completed rev 1:
- layout
- routing all trace
- ground fill
- silk screen art :)
Parts:
- MX16: footprint MX_Only:MXOnly-1U-NoLED -> MX_Only:MXOnly-2U-ReversedStabilizers-NoLED
Connections:
- net COL0: now also U1.8 (P0.24)
- net COL1: now also U1.7 (P0.22)
- net COL2: now also U1.6 (P0.20)
- net COL3: now also U1.5 (P0.17)
- net ROW0: now also U1.13 (NFC1/P0.09)
- net ROW1: now also U1.14 (NFC2/P0.10)
- net ROW2: now also U1.15 (P1.11)
- net ROW3: now also U1.16 (P1.13); no longer D15.1 (K)
- net ROW4: now also D15.1 (K), U1.17 (P1.15)
Changed lines of the file:
@@
 F 0 "MX16" H 5983 5323 60  0000 C CNN
 F 1 "MX-NoLED" H 5983 5249 20  0000 C CNN
-F 2 "MX_Only:MXOnly-1U-NoLED" H 5325 5075 60  0001 C CNN
+F 2 "MX_Only:MXOnly-2U-ReversedStabilizers-NoLED" H 5325 5075 60  0001 C CNN
 F 3 "" H 5325 5075 60  0001 C CNN
 	1    5950 5100
@@
 Wire Wire Line
 	6150 3950 5550 3950
-Wire Wire Line
-	7200 4750 6750 4750
 Connection ~ 5550 4750
 Wire Wire Line
@@
 Wire Wire Line
 	6150 4750 5550 4750
-Connection ~ 6750 4750
 Wire Wire Line
 	6750 4750 6150 4750
@@
 Wire Wire Line
 	7700 3100 7700 4700
+Connection ~ 6750 5550
 Wire Wire Line
-	7350 5200 7200 5200
+	7350 5200 7350 5550
 Wire Wire Line
-	7200 5200 7200 4750
+	6750 5550 7350 5550
+Text GLabel 4350 3850 2    50   Input ~ 0
+ROW0
+Text GLabel 4350 3750 2    50   Input ~ 0
+ROW1
+Text GLabel 4350 3650 2    50   Input ~ 0
+ROW2
+Text GLabel 4350 3550 2    50   Input ~ 0
+ROW3
+Text GLabel 4350 3450 2    50   Input ~ 0
+ROW4
+Text GLabel 2950 3450 0    50   Input ~ 0
+COL0
+Text GLabel 2950 3350 0    50   Input ~ 0
+COL1
+Text GLabel 2950 3250 0    50   Input ~ 0
+COL2
+Text GLabel 2950 3150 0    50   Input ~ 0
+COL3
 $EndSCHEMATC
