File: Choc corne/Choc corne.kicad_pcb (KiCad board)
At the start: 2 copper layers, 43 parts, among them U1 ProMicro

Commit message: big update
whatever
Parts:
- added D22: CD4148W, Diode_SMD:D_0805_2012Metric, F.Cu at (196.1, 151.6)
- added D23: CD4148W, Diode_SMD:D_0805_2012Metric, F.Cu at (258.5, 147.4)
- added D24: CD4148W, Diode_SMD:D_0805_2012Metric, F.Cu at (240.5, 164.9)
- added D25: CD4148W, Diode_SMD:D_0805_2012Metric, F.Cu at (228.8, 176.6)
- added D26: CD4148W, Diode_SMD:D_0805_2012Metric, F.Cu at (268.0, 138.4)
- added D27: CD4148W, Diode_SMD:D_0805_2012Metric, F.Cu at (269.6, 133.1)
- added D28: CD4148W, Diode_SMD:D_0805_2012Metric, F.Cu at (269.1, 130.1)
- added D29: CD4148W, Diode_SMD:D_0805_2012Metric, F.Cu at (264.6, 130.1)
- added D30: CD4148W, Diode_SMD:D_0805_2012Metric, F.Cu at (228.8, 173.5)
- added D31: CD4148W, Diode_SMD:D_0805_2012Metric, F.Cu at (228.8, 170.5)
- added D32: CD4148W, Diode_SMD:D_0805_2012Metric, F.Cu at (236.0, 167.9)
- added D33: CD4148W, Diode_SMD:D_0805_2012Metric, F.Cu at (236.0, 164.9)
- added D34: CD4148W, Diode_SMD:D_0805_2012Metric, F.Cu at (240.5, 161.8)
- added D35: CD4148W, Diode_SMD:D_0805_2012Metric, F.Cu at (236.0, 161.8)
- added D36: CD4148W, Diode_SMD:D_0805_2012Metric, F.Cu at (244.9, 158.8)
- added D37: CD4148W, Diode_SMD:D_0805_2012Metric, F.Cu at (240.5, 158.8)
- added D38: CD4148W, Diode_SMD:D_0805_2012Metric, F.Cu at (236.0, 158.8)
- added D39: CD4148W, Diode_SMD:D_0805_2012Metric, F.Cu at (247.4, 155.1)
- added D40: CD4148W, Diode_SMD:D_0805_2012Metric, F.Cu at (209.4, 151.6)
- added D41: CD4148W, Diode_SMD:D_0805_2012Metric, F.Cu at (205.0, 151.6)
- added D42: CD4148W, Diode_SMD:D_0805_2012Metric, F.Cu at (200.5, 151.6)
- added J1: MJ-4PP-9, Keebio-Parts:TRRS-PJ-320A, F.Cu at (146.1, 101.6)
- added J2: MJ-4PP-9, Keebio-Parts:TRRS-PJ-320A, F.Cu at (161.9, 101.6)
- added MX22: MX-NoLED, kbd:CherryMX_ChocV2_1u, F.Cu at (188.9, 69.8)
- added MX23: MX-NoLED, kbd:CherryMX_ChocV2_1u, F.Cu at (208.0, 67.5)
- added MX24: MX-NoLED, kbd:CherryMX_ChocV2_1u, F.Cu at (227.0, 65.1)
- added MX25: MX-NoLED, kbd:CherryMX_ChocV2_1u, F.Cu at (246.1, 67.5)
- added MX26: MX-NoLED, kbd:CherryMX_ChocV2_1u, F.Cu at (265.1, 72.2)
- added MX27: MX-NoLED, kbd:CherryMX_ChocV2_1u, F.Cu at (284.2, 72.2)
- added MX28: MX-NoLED, kbd:CherryMX_ChocV2_1u, F.Cu at (188.9, 88.9)
- added MX29: MX-NoLED, kbd:CherryMX_ChocV2_1u, F.Cu at (208.0, 86.5)
- added MX30: MX-NoLED, kbd:CherryMX_ChocV2_1u, F.Cu at (227.0, 84.1)
- added MX31: MX-NoLED, kbd:CherryMX_ChocV2_1u, F.Cu at (246.1, 86.5)
- added MX32: MX-NoLED, kbd:CherryMX_ChocV2_1u, F.Cu at (265.1, 91.3)
- added MX33: MX-NoLED, kbd:CherryMX_ChocV2_1u, F.Cu at (284.2, 91.3)
- added MX34: MX-NoLED, kbd:CherryMX_ChocV2_1u, F.Cu at (188.9, 108.0)
- added MX35: MX-NoLED, kbd:CherryMX_ChocV2_1u, F.Cu at (208.0, 105.6)
- added MX36: MX-NoLED, kbd:CherryMX_ChocV2_1u, F.Cu at (227.0, 103.2)
- added MX37: MX-NoLED, kbd:CherryMX_ChocV2_1u, F.Cu at (246.1, 105.6)
- added MX38: MX-NoLED, kbd:CherryMX_ChocV2_1u, F.Cu at (265.1, 110.3)
- added MX39: MX-NoLED, kbd:CherryMX_ChocV2_1u, F.Cu at (284.2, 110.3)
- added MX40: MX-NoLED, kbd:CherryMX_ChocV2_1.5u, F.Cu at (172.2, 137.3)
- added MX41: MX-NoLED, kbd:CherryMX_ChocV2_1u, F.Cu at (195.3, 132.6)
- added MX42: MX-NoLED, kbd:CherryMX_ChocV2_1u, F.Cu at (217.5, 129.4)
- added OL1: OLED, kbd:OLED_1side, F.Cu at (136.8, 95.1)
- added OL2: OLED, kbd:OLED_1side, F.Cu at (163.6, 95.1)
- added SW1: SW_PUSH, kbd:ResetSW_1side, F.Cu at (146.1, 115.1)
- added SW2: SW_PUSH, kbd:ResetSW_1side, F.Cu at (160.3, 115.1)
- added U2: Elite-C, Keebio-Parts:Elite-C, F.Cu at (167.5, 77.8)
- MX1, MX10, MX11, MX12, MX13, MX14, MX15, MX16, MX17, MX18, MX19, MX2, MX20, MX3, MX4, MX5, MX6, MX7, MX8, MX9: footprint Keebio-Parts:Kailh-PG1350-1u-NoLED -> kbd:CherryMX_ChocV2_1u
- MX21: footprint Keebio-Parts:Kailh-PG1350-1.5u -> kbd:CherryMX_ChocV2_1.5u
- U1: value ProMicro -> Elite-C; footprint Keebio-Parts:Elite-C-ZigZag -> Keebio-Parts:Elite-C; moved to F.Cu
- moved D1 153.7 mm to (39.7, 135.7)
- moved D10 153.7 mm to (30.8, 135.7)
- moved D12 153.7 mm to (17.4, 135.7)
- moved D14 153.7 mm to (48.6, 137.7)
- moved D15 153.7 mm to (53.0, 137.7)
- moved D17 153.7 mm to (61.9, 137.7)
- moved D18 153.7 mm to (48.6, 134.7)
- moved D19 153.7 mm to (53.0, 134.7)
- moved D2 153.7 mm to (21.9, 138.8)
- moved D21 153.7 mm to (61.9, 134.7)
- moved D3 153.7 mm to (26.3, 138.8)
- moved D4 153.7 mm to (21.9, 135.7)
- moved D5 153.7 mm to (30.8, 138.8)
- moved D7 153.7 mm to (39.7, 138.8)
- moved D9 153.7 mm to (26.3, 135.7)
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Connections:
- net Net-(U1-Pad2) renamed DATA
- U1 pad 21: Net-(U1-Pad21) -> VCC
- U1 pad 22: Net-(U1-Pad22) -> RESET
- U1 pad 23: Net-(U1-Pad23) -> GND
- U1 pad 3: Net-(U1-Pad3) -> GND
- U1 pad 4: Net-(U1-Pad4) -> GND
- U1 pad 5: Net-(U1-Pad5) -> SDA
- U1 pad 6: Net-(U1-Pad6) -> SCL

Commit message: Added partial pcb routing
Parts:
- D22, D23, D24, D25, D26, D27, D28, D29, D30, D31, D32, D33, D34, D35, D36, D37, D38, D39, D40, D41, D42: moved to B.Cu
- moved D12 119.2 mm to (127.0, 88.9), turned to 90 degrees
- moved D6 114.7 mm to (127.0, 70.0), turned to 90 degrees
- moved D25 111.8 mm to (254.0, 67.6), turned to 90 degrees
- moved D5 105.0 mm to (108.0, 67.6), turned to 90 degrees
- moved D24 99.8 mm to (234.9, 65.2), turned to 90 degrees
- moved D4 97.3 mm to (88.9, 65.2), turned to 90 degrees
- moved D33 92.4 mm to (292.1, 91.4), turned to 90 degrees
- moved D23 90.4 mm to (215.9, 67.6), turned to 90 degrees
- moved D30 89.4 mm to (234.9, 84.3), turned to 90 degrees
- moved D11 87.7 mm to (108.0, 86.7), turned to 90 degrees
- moved D31 87.5 mm to (254.0, 86.7), turned to 90 degrees
- moved D32 85.0 mm to (273.1, 91.4), turned to 90 degrees
- moved D3 83.4 mm to (69.8, 67.6), turned to 90 degrees
- moved D28 83.1 mm to (196.8, 88.9), turned to 90 degrees
- moved D18 82.8 mm to (127.0, 108.1), turned to 90 degrees
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Connections:
- U1 pad 10: Net-(U1-Pad10) -> ROW3
- U1 pad 7: Net-(U1-Pad7) -> ROW0
- U1 pad 8: Net-(U1-Pad8) -> ROW1
- U1 pad 9: Net-(U1-Pad9) -> ROW2
Routing:
- net ROW2: track 0.00 -> 169.1 mm
- net ROW1: track 0.00 -> 154.6 mm
- net ROW0: track 0.00 -> 152.0 mm
- net ROW3: track 0.00 -> 124.9 mm
- net GND: track 0.00 -> 105.0 mm
- net COL5: track 0.00 -> 93.4 mm
- net COL7: track 0.00 -> 85.1 mm
- net COL4: track 0.00 -> 84.0 mm
- net COL6: track 0.00 -> 83.8 mm
- net COL3: track 0.00 -> 83.7 mm
- net COL8: track 0.00 -> 82.6 mm
- net COL11: track 0.00 -> 51.2 mm
- net COL10: track 0.00 -> 51.2 mm
- net COL0: track 0.00 -> 51.2 mm
- net COL2: track 0.00 -> 51.2 mm
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