File: Corne Integrated Microchip/Corne Integrated Microchip.sch (KiCad schematic (older format))
At the start: 44 parts, among them J1 MJ-4PP-9, J2 MJ-4PP-9, SW1 SW_Push, SW2 SW_Push, U1 ATmega32U4-AU, U2 ATmega32U4-AU, U3 PRTR5V0U2X, U4 PRTR5V0U2X, Y1 16MHz, Y2 16MHz

Commit message: Assigned Footprint
Parts:
- C1, C10, C11, C12, C13, C14, C15, C16, C2, C3, C4, C5, C6, C7, C8, C9: footprint (none) -> Capacitor_SMD:C_0805_2012Metric_Pad1.15x1.40mm_HandSolder
- F1, F2: footprint (none) -> Fuse:Fuse_1206_3216Metric_Pad1.42x1.75mm_HandSolder
- J1, J2: footprint (none) -> kbd:MJ-4PP-9_1side
- OL1, OL2: footprint (none) -> kbd:OLED_1side
- R1, R10, R11, R12, R2, R3, R4, R5, R6, R7, R8, R9: footprint (none) -> Resistor_SMD:R_0805_2012Metric_Pad1.15x1.40mm_HandSolder
- SW1, SW2: footprint (none) -> kbd:ResetSW_1side
- U3, U4: footprint (none) -> random-keyboard-parts:SOT143B
- USB1, USB2: footprint (none) -> Type-C:HRO-TYPE-C-31-M-12-HandSoldering
- Y1, Y2: footprint (none) -> Crystal:Crystal_SMD_3225-4Pin_3.2x2.5mm_HandSoldering
Connections:
- net +5V: no longer F1.1
- net +5VA: now also F1.1
- net D+: no longer R6.1
- net D-: no longer R5.1
- net GND: no longer R7.1, R8.1, U3.1 (GND), USB1.1 (GND), USB1.12 (GND), USB1.13 (SHIELD)
- net GNDA: now also R7.1, R8.1, U3.1 (GND), USB1.1 (GND), USB1.12 (GND), USB1.13 (SHIELD)
- net VCC: no longer F1.2, U3.4 (VCC), USB1.11 (VBUS), USB1.2 (VBUS)
- net VDD: now also F1.2, U3.4 (VCC), USB1.11 (VBUS), USB1.2 (VBUS)
- net D-_R: now reaches U2.3 (D-)
- net D-_R: now also R5.1
- net D+_R: now reaches U2.4 (D+)
- net D+_R: now also R6.1
- no-connect marks 10 -> 8
