File: Corne Integrated Microchip/matrix.sch (KiCad schematic (older format))
At the start: 84 parts

Commit message: Assigned Footprint
Parts:
- D1, D10, D11, D12, D13, D14, D15, D16, D17, D18, D19, D2, D20, D21, D22, D23, D24, D25, D26, D27, D28, D29, D3, D30, D31, D32, D33, D34, D35, D36, D37, D38, D39, D4, D40, D41, D42, D5, D6, D7, D8, D9: footprint (none) -> Diode_SMD:D_SOD-123
- MX1, MX10, MX11, MX12, MX13, MX14, MX15, MX16, MX17, MX18, MX19, MX2, MX20, MX22, MX23, MX24, MX25, MX26, MX27, MX28, MX29, MX3, MX30, MX31, MX32, MX33, MX34, MX35, MX36, MX37, MX38, MX39, MX4, MX41, MX42, MX5, MX6, MX7, MX8, MX9: footprint (none) -> kbd:CherryMX_ChocV2_1u
- MX21, MX40: footprint (none) -> kbd:CherryMX_ChocV2_1.5u

Commit message: Started routing
Connections:
- net ROW3: now also D19.1 (K), D20.1 (K), D21.1 (K); no longer D13.1 (K), D14.1 (K), D15.1 (K), D16.1 (K), D17.1 (K), D18.1 (K)
- net ROW4: no longer D19.1 (K), D20.1 (K), D21.1 (K)
- new net ROW2: D13.1 (K), D14.1 (K), D15.1 (K), D16.1 (K), D17.1 (K), D18.1 (K)
Changed lines of the file:
@@
 EESchema Schematic File Version 4
+LIBS:Corne Integrated Microchip-cache
 EELAYER 30 0
 EELAYER END
@@
 COL0
 Text GLabel 3100 5250 0    50   Input ~ 0
-ROW4
+ROW3
 Text GLabel 1600 4600 0    50   Input ~ 0
-ROW3
+ROW2
 Text GLabel 1600 3950 0    50   Input ~ 0
 ROW1
