File: Corne Integrated Microchip/Corne Integrated Microchip.kicad_pcb (KiCad board)
At the start: 2 copper layers, 128 parts, among them J1 MJ-4PP-9, J2 MJ-4PP-9, SW1 SW_Push, SW2 SW_Push, U1 ATmega32U4-AU, U2 ATmega32U4-AU, U3 PRTR5V0U2X, U4 PRTR5V0U2X, Y1 16MHz, Y2 16MHz

Commit message: Started routing
Parts:
- C1, C10, C11, C12, C13, C14, C15, C16, C2, C3, C4, C5, C6, C7, C8, C9, F1, F2, J1, J2, OL1, OL2, R1, R10, R11, R12, R2, R3, R4, R5, R6, R7, R8, R9, SW1, SW2, U1, U2, U3, U4, USB1, USB2, Y1, Y2: moved to F.Cu
- moved D26 215.7 mm to (264.3, 58.0), turned to 90 degrees
- moved MX1 207.6 mm to (21.4, 57.9)
- moved D27 207.0 mm to (267.5, 58.0), turned to 90 degrees
- moved D38 204.2 mm to (264.3, 96.1), turned to 90 degrees
- moved D33 200.9 mm to (267.5, 77.1), turned to 90 degrees
- moved D32 197.2 mm to (264.3, 77.1), turned to 90 degrees
- moved MX39 189.6 mm to (275.4, 96.0)
- moved D39 181.4 mm to (267.5, 96.1), turned to 90 degrees
- moved D25 175.7 mm to (229.4, 52.4), turned to 90 degrees
- moved D42 175.6 mm to (216.7, 111.2), turned to 90 degrees
- moved D24 174.7 mm to (226.2, 52.4), turned to 90 degrees
- moved D37 171.2 mm to (229.4, 90.5), turned to 90 degrees
- moved D31 169.2 mm to (229.4, 71.5), turned to 90 degrees
- moved D40 165.2 mm to (196.1, 111.1), turned to 90 degrees
- moved D36 163.1 mm to (226.2, 90.5), turned to 90 degrees
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Connections:
- D13 pad 1: ROW3 -> ROW2
- D14 pad 1: ROW3 -> ROW2
- D15 pad 1: ROW3 -> ROW2
- D16 pad 1: ROW3 -> ROW2
- D17 pad 1: ROW3 -> ROW2
- D18 pad 1: ROW3 -> ROW2
- D19 pad 1: ROW4 -> ROW3
- D20 pad 1: ROW4 -> ROW3
- D21 pad 1: ROW4 -> ROW3
Other:
- board outline added: 273.1 x 94.5 mm

Commit message: continued routing
Parts:
- OL1, OL2: footprint kbd:OLED_1side -> kbd:OLED
- moved USB1 133.5 mm to (160.3, 41.3), turned to 180 degrees
- moved OL1 112.4 mm to (133.3, 92.1)
- moved C11 110.5 mm to (146.1, 80.2), turned to 225 degrees
- moved C9 103.8 mm to (128.6, 80.2), turned to 135 degrees
- moved C10 94.8 mm to (139.0, 66.7), turned to 135 degrees
- moved R1 91.9 mm to (136.5, 63.6), turned to 225 degrees
- moved C8 91.4 mm to (140.4, 85.7), turned to 45 degrees
- moved C7 82.8 mm to (146.4, 74.5), turned to 135 degrees
- moved R3 74.4 mm to (133.3, 84.9), turned to 315 degrees
- moved OL2 45.3 mm to (32.5, 148.4)
- moved U2 18.2 mm to (71.4, 142.9)
- moved R10 10.1 mm to (135.7, 58.7), turned to 90 degrees
- moved R9 10.1 mm to (138.9, 58.7), turned to 90 degrees
- moved C5 7.21 mm to (142.1, 69.8), turned to 315 degrees
- moved Y1 4.92 mm to (130.5, 58.6), turned to 330 degrees
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Connections:
- U1 pad 18: Net-(U1-Pad18) -> ROW0
- U1 pad 19: Net-(U1-Pad19) -> ROW1
- U1 pad 20: Net-(U1-Pad20) -> ROW2
- U1 pad 21: Net-(U1-Pad21) -> ROW3
Routing:
- net GND: track 0.00 -> 164.4 mm, vias 0 -> 6
- net ROW0: track 0.00 -> 91.5 mm
- net ROW1: track 0.00 -> 91.1 mm
- net ROW2: track 0.00 -> 88.4 mm
- net COL5: track 0.00 -> 85.9 mm
- net COL4: track 0.00 -> 77.4 mm
- net COL3: track 0.00 -> 76.6 mm
- net VCC: track 0.00 -> 76.0 mm, vias 0 -> 4
- net +5V: track 0.00 -> 71.8 mm, vias 0 -> 2
- net COL0: track 0.00 -> 49.1 mm
- net COL2: track 0.00 -> 48.8 mm
- net COL1: track 0.00 -> 48.8 mm
- net DATA: track 0.00 -> 46.6 mm, vias 0 -> 2
- net Net-(D21-Pad2): track 0.00 -> 43.0 mm
- net Net-(R1-Pad2): track 0.00 -> 35.0 mm, vias 0 -> 2
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Other:
- board size 273.1 x 94.5 mm -> 273.8 x 94.5 mm

Commit message: Finished routing
Parts:
- moved OL2 136.4 mm to (156.7, 92.1)
- moved R5 130.3 mm to (161.9, 59.0), turned to 90 degrees
- moved R2 129.6 mm to (159.5, 63.5), turned to 225 degrees
- moved C4 128.9 mm to (156.0, 64.1), turned to 270 degrees
- moved R8 128.6 mm to (165.1, 54.0), turned to 180 degrees
- moved C15 127.5 mm to (161.9, 66.7), turned to 135 degrees
- moved F1 124.6 mm to (166.7, 58.6), turned to 90 degrees
- moved C12 122.8 mm to (169.4, 74.7), turned to 135 degrees
- moved U3 116.7 mm to (160.3, 54.0)
- moved R6 116.1 mm to (158.8, 59.0), turned to 90 degrees
- moved U2 110.7 mm to (160.3, 77.0), turned to 225 degrees
- moved C6 108.8 mm to (165.1, 69.8), turned to 315 degrees
- moved R7 106.8 mm to (155.3, 54.0)
- moved Y2 102.9 mm to (153.5, 58.6), turned to 330 degrees
- moved R4 102.0 mm to (156.4, 84.9), turned to 315 degrees
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Connections:
- U1 pad 36: Net-(U1-Pad36) -> COL5
- U1 pad 37: Net-(U1-Pad37) -> COL4
- U1 pad 38: Net-(U1-Pad38) -> COL3
- U1 pad 39: Net-(U1-Pad39) -> COL2
- U1 pad 40: Net-(U1-Pad40) -> COL1
- U1 pad 41: Net-(U1-Pad41) -> COL0
- U2 pad 25: Net-(U2-Pad25) -> COL11
- U2 pad 26: Net-(U2-Pad26) -> COL10
- U2 pad 27: Net-(U2-Pad27) -> COL9
- U2 pad 28: Net-(U2-Pad28) -> COL8
- U2 pad 29: Net-(U2-Pad29) -> COL7
- U2 pad 30: Net-(U2-Pad30) -> COL6
- U2 pad 38: Net-(U2-Pad38) -> ROW7
- U2 pad 39: Net-(U2-Pad39) -> ROW6
- U2 pad 40: Net-(U2-Pad40) -> ROW5
- U2 pad 41: Net-(U2-Pad41) -> ROW4
Routing:
- net GNDA: track 0.00 -> 230.4 mm, vias 0 -> 12
- net COL11: track 0.00 -> 221.4 mm
- net COL10: track 0.00 -> 200.9 mm
- net COL0: track 49.1 -> 241.1 mm, vias 0 -> 2
- net COL9: track 0.00 -> 182.5 mm
- net COL1: track 48.8 -> 218.1 mm
- net COL8: track 0.00 -> 167.5 mm
- net COL7: track 0.00 -> 152.8 mm
- net COL2: track 48.8 -> 198.0 mm
- net ROW4: track 0.00 -> 132.4 mm, vias 0 -> 1
- net ROW6: track 0.00 -> 130.6 mm, vias 0 -> 1
- net ROW5: track 0.00 -> 121.5 mm, vias 0 -> 1
- net COL6: track 0.00 -> 114.1 mm
- net COL3: track 76.6 -> 186.5 mm
- net COL4: track 77.4 -> 163.4 mm
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- added copper zone on B.Cu, net GND
- added copper zone on F.Cu, net GND
- added copper zone on B.Cu, net GNDA
- added copper zone on F.Cu, net GNDA

Commit message: Optimizing optimizing optimizing
Parts:
- moved R6 5.33 mm to (164.1, 59.0)
- moved C13 4.76 mm to (168.3, 85.7)
- moved C14 4.76 mm to (156.4, 80.2)
- moved C2 4.76 mm to (158.0, 64.1)
- moved C4 4.76 mm to (160.7, 64.1)
- moved C6 4.76 mm to (169.9, 69.8)
- moved D22 4.76 mm to (193.7, 54.0)
- moved D24 4.76 mm to (231.8, 52.4)
- moved D28 4.76 mm to (193.7, 73.1)
- moved D30 4.76 mm to (231.8, 71.5)
- moved D34 4.76 mm to (193.7, 92.1)
- moved D36 4.76 mm to (231.8, 90.5)
- moved D40 4.76 mm to (201.6, 111.1)
- moved MX22 4.76 mm to (185.7, 55.6)
- moved MX24 4.76 mm to (223.8, 50.8)
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Connections:
- net D+_R renamed rD+
- net D-_R renamed rD-
- net Net-(R10-Pad2) renamed DP
- net Net-(R5-Pad2) renamed rDN
- net Net-(R6-Pad2) renamed rDP
- net Net-(R9-Pad2) renamed DN
Routing:
- net +5V: track 79.3 -> 95.9 mm, vias 2 -> 4
- net GNDA: track 230.4 -> 246.1 mm, vias 12 -> 15
- net +5VA: track 83.1 -> 97.2 mm, vias 2 -> 6
- net VCC: track 76.7 -> 72.4 mm, vias 4 -> 2
- net rDP: track 13.4 -> 12.2 mm
- net DP: track 13.2 -> 12.0 mm
- net Net-(C3-Pad1): track 15.5 -> 16.5 mm
- net rD+: track 18.5 -> 17.9 mm
- net D+: track 18.9 -> 18.4 mm
- net Net-(C4-Pad1): track 15.7 -> 16.2 mm
Other:
- board size 273.8 x 94.5 mm -> 282.6 x 94.5 mm

Commit message: Final? rev 1.0
Tidied everything up, should be good to go now :)
Parts:
- added G***: LOGO, pcb-art:martinwithball, F.Cu at (68.3, 106.4)
- moved R2 28.0 mm to (173.8, 89.8), turned to 180 degrees
- moved R1 27.4 mm to (125.3, 90.0), turned to 180 degrees
- moved C15 2.25 mm to (165.1, 65.1), turned to 90 degrees
- moved C10 2.19 mm to (133.3, 65.3), turned to 90 degrees
Routing:
- net GNDA: track 246.1 -> 171.5 mm, vias 15 -> 8
- net GND: track 218.8 -> 169.8 mm, vias 11 -> 7
- net Net-(R2-Pad2): track 53.6 -> 33.2 mm, vias 1 -> 2
- net Net-(R1-Pad2): track 35.0 -> 26.8 mm
- net +5VA: track 97.2 -> 98.8 mm
- net COL0: track 241.1 -> 239.5 mm, vias 2 -> 0
- net COL5: track 135.5 -> 134.6 mm
- net COL1: track 218.1 -> 217.3 mm
- net COL2: track 198.0 -> 197.3 mm
- net COL3: track 186.5 -> 185.7 mm
- net COL4: track 163.4 -> 162.7 mm
- net DATA: track 42.7 -> 42.2 mm
Other:
- board text added: "honk40 designed by evan"

Commit message: Added breakaway tabs
Added breakaway tabs to connect both sides of the board.
Parts:
- added J5: Breakaway_Tabs, kbd:Breakaway_Tabs, F.Cu at (93.7, 43.7)
- added J5: Breakaway_Tabs, kbd:Breakaway_Tabs, F.Cu at (55.6, 43.7)
- added REF**: Breakaway_Tabs, kbd:Breakaway_Tabs, F.Cu at (27.0, 105.6)
- added REF**: Breakaway_Tabs, kbd:Breakaway_Tabs, F.Cu at (267.5, 105.6)
- added REF**: Breakaway_Tabs, kbd:Breakaway_Tabs, F.Cu at (238.9, 43.7)
- added REF**: Breakaway_Tabs, kbd:Breakaway_Tabs, F.Cu at (200.8, 43.7)
- moved C12 3.97 mm to (170.2, 74.7)
- moved C13 3.97 mm to (164.3, 85.7)
- moved C14 3.97 mm to (152.4, 80.2)
- moved C15 3.97 mm to (161.1, 65.1)
- moved C16 3.97 mm to (170.1, 80.2)
- moved C2 3.97 mm to (154.0, 64.1)
- moved C4 3.97 mm to (156.7, 64.1)
- moved C6 3.97 mm to (165.9, 69.8)
- moved D22 3.97 mm to (189.7, 54.0)
- moved D23 3.97 mm to (192.9, 54.0)
- moved D24 3.97 mm to (227.8, 52.4)
- moved D25 3.97 mm to (231.0, 52.4)
- moved D26 3.97 mm to (265.9, 58.0)
- moved D27 3.97 mm to (269.1, 58.0)
- moved D28 3.97 mm to (189.7, 73.1)
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Other:
- board size 282.6 x 94.5 mm -> 278.6 x 103.2 mm
